Commit message: add meshes to b2piper & fix isaacgym robot 关节错位

File: low-level/resources/robots/b2piper/urdf/b2_piper.urdf (robot description, URDF)
Before this commit: robot b2_piper_description, 47 links, 46 joints
Links:
- link FL_calf: geometry collision box size=0.05 0.028 0.035; collision box size=0.1 0.0245 0.018
- link FL_hip: geometry collision cylinder length=0.05 radius=0.07; visual mesh filename=../meshes/FL_hip.dae
- link FL_thigh: geometry collision box size=0.32 0.0445 0.054; visual mesh filename=../meshes/FL_thigh.dae
- link FR_calf: geometry collision box size=0.05 0.028 0.035; collision box size=0.1 0.0245 0.018
- link FR_hip: geometry collision cylinder length=0.05 radius=0.07; visual mesh filename=../meshes/FR_hip.dae
- link FR_thigh: geometry collision box size=0.25 0.028 0.04; visual mesh filename=../meshes/FR_thigh.dae
- link RL_calf: geometry collision box size=0.05 0.028 0.035; collision box size=0.1 0.0245 0.018
- link RL_hip: geometry collision cylinder length=0.05 radius=0.07; visual mesh filename=../meshes/RL_hip.dae
- link RL_thigh: geometry collision box size=0.25 0.028 0.04; visual mesh filename=../meshes/RL_thigh.dae
- link RR_calf: geometry collision box size=0.05 0.028 0.035; collision box size=0.1 0.0245 0.018
- link RR_hip: geometry collision cylinder length=0.05 radius=0.07; visual mesh filename=../meshes/RR_hip.dae
- link RR_thigh: geometry collision box size=0.25 0.028 0.04; visual mesh filename=../meshes/RR_thigh.dae
- link arm_base: geometry collision mesh filename=../meshes/base_link.STL; visual mesh filename=../meshes/base_link.STL
- link arm_link1: geometry collision mesh filename=../meshes/link1.STL; visual mesh filename=../meshes/link1.STL
- link arm_link2: geometry collision mesh filename=../meshes/link2.STL; visual mesh filename=../meshes/link2.STL
- link arm_link3: geometry collision mesh filename=../meshes/link3.STL; visual mesh filename=../meshes/link3.STL
- link arm_link4: geometry collision mesh filename=../meshes/link4.STL; visual mesh filename=../meshes/link4.STL
- link arm_link5: geometry collision mesh filename=../meshes/link5.STL; visual mesh filename=../meshes/link5.STL
- link arm_link6: geometry collision mesh filename=../meshes/link6.STL; visual mesh filename=../meshes/link6.STL
- link arm_link7: geometry collision mesh filename=../meshes/link7.STL; visual mesh filename=../meshes/link7.STL
- link arm_link8: geometry collision mesh filename=../meshes/link8.STL; visual mesh filename=../meshes/link8.STL
- link base_link: geometry collision box size=0.5 0.28 0.15; visual mesh filename=../meshes/base_link.dae
- link gripper_base: geometry collision mesh filename=../meshes/gripper_base.STL; visual mesh filename=../meshes/gripper_base.STL

Commit message: fix isaacgym robot visualize

File: low-level/resources/robots/b2piper/urdf/b2_piper.urdf (robot description, URDF)
Before this commit: robot b2_piper_description, 47 links, 46 joints
Links:
- link FL_calf: geometry collision box size=0.05 0.028 0.035; collision box size=0.1 0.0245 0.018
- link FL_hip: geometry collision cylinder length=0.05 radius=0.07; visual mesh filename=../meshes_b2_ig_false/FL_hip.dae
- link FL_thigh: geometry collision box size=0.32 0.0445 0.054; visual mesh filename=../meshes_b2_ig_false/FL_thigh.dae
- link FR_calf: geometry collision box size=0.05 0.028 0.035; collision box size=0.1 0.0245 0.018
- link FR_hip: geometry collision cylinder length=0.05 radius=0.07; visual mesh filename=../meshes_b2_ig_false/FR_hip.dae
- link FR_thigh: geometry collision box size=0.25 0.028 0.04; visual mesh filename=../meshes_b2_ig_false/FR_thigh.dae
- link RL_calf: geometry collision box size=0.05 0.028 0.035; collision box size=0.1 0.0245 0.018
- link RL_hip: geometry collision cylinder length=0.05 radius=0.07; visual mesh filename=../meshes_b2_ig_false/RL_hip.dae
- link RL_thigh: geometry collision box size=0.25 0.028 0.04; visual mesh filename=../meshes_b2_ig_false/RL_thigh.dae
- link RR_calf: geometry collision box size=0.05 0.028 0.035; collision box size=0.1 0.0245 0.018
- link RR_hip: geometry collision cylinder length=0.05 radius=0.07; visual mesh filename=../meshes_b2_ig_false/RR_hip.dae
- link RR_thigh: geometry collision box size=0.25 0.028 0.04; visual mesh filename=../meshes_b2_ig_false/RR_thigh.dae
- link base_link: geometry collision box size=0.5 0.28 0.15; visual mesh filename=../meshes_b2_ig_false/base_link.dae
